File: wheel.kicad_sch (KiCad schematic)
At the start: 9 parts, among them J1 Conn_01x09, SW1 SW_DPST, SW2 SW_DPST, SW3 SW_DPST, SW4 SW_DPST, SW5 SW_DPST, SW6 SW_DPST, SW7 SW_DPST, SW8 SW_DPST

Commit message: add firmware
Parts:
- removed J1: Conn_01x09, Connector_PinHeader_2.54mm:PinHeader_1x09_P2.54mm_Vertical, symbol Connector_Generic:Conn_01x09
- removed SW1, SW2, SW3, SW4, SW5, SW6, SW7, SW8: SW_DPST, Button_Switch_THT:SW_PUSH_6mm, symbol Switch:SW_DPST
Other:
- added sheet Buttons (buttons.kicad_sch)
- added sheet encoder_board (encoder.kicad_sch)
